File: sensor-pcb/sensor-pcb.kicad_sch (KiCad schematic)
At the start: 15 parts, among them J1 Conn_01x03, J2 Conn_01x02, J3 Conn_01x01_Socket, J4 Conn_01x01_Socket, Q2 BSS84, U1 TLV9151IDBVR

Commit message: Fix flipped power pins
Connections:
- net GND: now also J1.3 (Pin_3); no longer J1.1 (Pin_1)
- net VIN: now also J1.1 (Pin_1); no longer J1.3 (Pin_3)
Changed lines of the file:
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@@
 		(lib_id "Connector_Generic:Conn_01x03")
 		(at 170.18 104.14 0)
-		(mirror x)
 		(unit 1)
 		(exclude_from_sim no)
@@
 		(dnp no)
 		(property "Reference" "J1"
-			(at 172.72 105.4101 0)
+			(at 172.72 102.8699 0)
 			(effects
 				(font
@@
 		)
 		(property "Value" "Conn_01x03"
-			(at 172.72 102.8701 0)
+			(at 172.72 105.4099 0)
 			(effects
 				(font

Commit message: Reverse direction
Connections:
- net +5V: now also RV1.3; no longer RV1.1
- net GND: now also RV1.1; no longer RV1.3
Changed lines of the file:
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@@
 		(lib_id "Device:R_Potentiometer")
 		(at 76.2 101.6 0)
+		(mirror x)
 		(unit 1)
 		(exclude_from_sim no)
@@
 		(on_board yes)
 		(dnp no)
-		(fields_autoplaced yes)
 		(property "Reference" "RV1"
-			(at 73.66 100.3299 0)
+			(at 73.66 102.8701 0)
 			(effects
 				(font
@@
 		)
 		(property "Value" "RDC503052A"
-			(at 73.66 102.8699 0)
+			(at 73.66 100.3301 0)
 			(effects
 				(font

Commit message: Change design to allow arbitrary polarity
Parts:
- removed Q2: BSS84, Package_TO_SOT_SMD:SOT-23, symbol Transistor_FET:BSS84
- added Q7: BSS84DW-7-F, Package_TO_SOT_SMD:SOT-363_SC-70-6, symbol Transistor_FET:Q_Dual_PMOS_S1G1D2S2G2D1
- added Q8: 2N7002DW, Package_TO_SOT_SMD:SOT-363_SC-70-6, symbol Transistor_FET:Q_Dual_NMOS_S1G1D2S2G2D1
Connections:
- net +5V: now also Q7.1 (S), Q7.4 (S); no longer RV1.3
- net GND: now also Q8.1 (S), Q8.4 (S); no longer J1.3 (Pin_3), RV1.1
- net VIN renamed VIN1
- net VIN1: now also RV1.3, Q7.5 (G), Q7.6 (D), Q8.5 (G), Q8.6 (D)
- new net VIN2: J1.3 (Pin_3), Q7.2 (G), Q7.3 (D), Q8.2 (G), Q8.3 (D), RV1.1
Other:
- moved on the sheet: C2, J1, J2, J3, J4
